Commit message: Launch fix

File: src/rover30_description/urdf/lidar.xacro (robot description, xacro)
@@ -5,5 +5,5 @@
         <parent link="base_link"/>
         <child link="laser_frame"/>
-        <origin xyz="11 0 10" rpy="0 0 0"/>
+        <origin xyz="11 0 15" rpy="0 0 0"/>
     </joint>
     <link name="laser_frame">
@@ -22,5 +22,5 @@
         </collision>
         <xacro:inertial_cylinder mass="0.1" length="1.0" radius="1.0">
-            <origin xyz="11 0 10" rpy="0 0 0"/>
+            <origin xyz="11 0 15" rpy="0 0 0"/>
         </xacro:inertial_cylinder>
     </link>
@@ -41,5 +41,5 @@
                 <range>
                     <min>0.3</min>
-                    <max>12</max>
+                    <max>25</max>
                 </range>
             </ray>

File: src/rover30_description/urdf/rover30_core.xacro (robot description, xacro)
@@ -4,9 +4,23 @@
     <link name="base_link">
         <visual>
-            <origin xyz="0 0 0" rpy="0 0 0"/>
+            <origin xyz="0 0 5" rpy="0 0 0"/>
             <geometry>
                 <mesh filename="package://rover30_description/meshes/rover_body.stl"/>
             </geometry>
         </visual>
+        <collision>
+            <origin xyz="0 0 5" rpy="0 0 0"/>
+            <geometry>
+                <mesh filename="package://rover30_description/meshes/rover_body.stl"/>
+            </geometry>
+        </collision>
+        <inertial>
+            <origin xyz="0 0 5" rpy="0 0 0"/>
+            <mass value="20.0"/>
+            <inertia
+            ixx="1.0" ixy="1.0" ixz="1.0"
+            iyy="1.0" iyz="1.0"
+            izz="1.0" />
+        </inertial>
      </link>
     <link name="right_front_wheel">
@@ -20,4 +34,18 @@
             </material>
         </visual>
+        <collision>
+            <origin xyz="6.25 -4.1 -1.5" rpy="0 0 0"/>
+            <geometry>
+                <mesh filename="package://rover30_description/meshes/kolo.stl" scale="2.0 2.0 2.0"/>
+            </geometry>
+        </collision>
+        <inertial>
+            <origin xyz="6.25 -4.1 -1.5" rpy="0 0 0"/>
+            <mass value="2.0"/>
+            <inertia
+              ixx="0.01" ixy="0.0" ixz="0.0"
+              iyy="0.01" iyz="0.0"
+              izz="0.01"/>
+          </inertial>
     </link>
     <link name="left_front_wheel">
@@ -31,4 +59,18 @@
             </material>
         </visual>
+        <collision>
+            <origin xyz="6.25 4.7 -1.5" rpy="0 0 0"/>
+            <geometry>
+                <mesh filename="package://rover30_description/meshes/kolo.stl" scale="2.0 2.0 2.0"/>
+            </geometry>
+        </collision>
+        <inertial>
+            <origin xyz="6.25 4.7 -1.5" rpy="0 0 0"/>
+            <mass value="2.0"/>
+            <inertia
+              ixx="0.01" ixy="0.0" ixz="0.0"
+              iyy="0.01" iyz="0.0"
+              izz="0.01"/>
+          </inertial>
     </link>
     <link name="right_rear_wheel">
@@ -42,4 +84,18 @@
             </material>
         </visual>
+        <collision>
+            <origin xyz="-2.6 -4.1 -1.5" rpy="0 0 0"/>
+            <geometry>
+                <mesh filename="package://rover30_description/meshes/kolo.stl" scale="2.0 2.0 2.0"/>
+            </geometry>
+        </collision>
+        <inertial>
+            <origin xyz="-2.6 -4.1 -1.5" rpy="0 0 0"/>
+            <mass value="2.0"/>
+            <inertia
+              ixx="0.01" ixy="0.0" ixz="0.0"
+              iyy="0.01" iyz="0.0"
+              izz="0.01"/>
+          </inertial>
     </link>
     <link name="left_rear_wheel">
@@ -53,29 +109,43 @@
             </material>
         </visual>
+        <collision>
+            <origin xyz="-2.6 4.7 -1.5" rpy="0 0 0"/>
+            <geometry>
+                <mesh filename="package://rover30_description/meshes/kolo.stl" scale="2.0 2.0 2.0"/>
+            </geometry>
+        </collision>
+        <inertial>
+            <origin xyz="-2.6 4.7 -1.5" rpy="0 0 0"/>
+            <mass value="2.0"/>
+            <inertia
+              ixx="0.01" ixy="0.0" ixz="0.0"
+              iyy="0.01" iyz="0.0"
+              izz="0.01"/>
+          </inertial>
     </link>
      <joint name="base_joint" type="fixed">
         <parent link="base_footprint"/>
         <child link="base_link"/>
-        <origin xyz="0 0 0.033" rpy="0 0 0"/>
+        <origin xyz="0 0 5.033" rpy="0 0 0"/>
      </joint>
-    <joint name="rww" type="fixed">
+    <joint name="rfw" type="fixed">
         <parent link="base_link"/>
         <child link="right_front_wheel"/>
-        <origin xyz="6.25 -4.1 -1.5" rpy="0 0 0"/>
+        <origin xyz="6.25 -4.1 3.5" rpy="0 0 0"/>
     </joint>
     <joint name="lfw" type="fixed">
         <parent link="base_link"/>
         <child link="left_front_wheel"/>
-        <origin xyz="6.25 4.7 -1.5" rpy="0 0 0"/>
+        <origin xyz="6.25 4.7 3.5" rpy="0 0 0"/>
     </joint>
     <joint name="rrw" type="fixed">
         <parent link="base_link"/>
         <child link="right_rear_wheel"/>
-        <origin xyz="-2.6 -4.1 -1.5" rpy="0 0 0"/>
+        <origin xyz="-2.6 -4.1 3.5" rpy="0 0 0"/>
     </joint>
     <joint name="lrw" type="fixed">
         <parent link="base_link"/>
         <child link="left_rear_wheel"/>
-        <origin xyz="-2.6 4.7 -1.5" rpy="0 0 0"/>
+        <origin xyz="-2.6 4.7 3.5" rpy="0 0 0"/>
     </joint>
 </robot>
