Commit message: sory, lidar tyl na przód był nie wiem czemu

File: src2/rover30_description/urdf/lidar.xacro (robot description, xacro)
@@ -5,5 +5,5 @@
         <parent link="base_link"/>
         <child link="laser_frame"/>
-        <origin xyz="-8.79607 0 6.3" rpy="0 0 0"/>
+        <origin xyz="8.79607 0 6.3" rpy="0 0 0"/>
     </joint>
     <link name="laser_frame">
@@ -22,5 +22,5 @@
         </collision>
         <xacro:inertial_cylinder mass="0.1" length="1.0" radius="1.0">
-            <origin xyz="-8.79607 0 6.3" rpy="0 0 0"/>
+            <origin xyz="8.79607 0 6.3" rpy="0 0 0"/>
         </xacro:inertial_cylinder>
     </link>
