Commit message: XUAZ is not rotating anymore, changed inertial properites of meshes, gazebo works

File: src2/rover30_description/urdf/interial_macros.xacro (robot description, xacro)
@@ -1,4 +1,4 @@
 <?xml version="1.0"?>
-<robot xmlns:xacro="http://ros.org/wiki/xacro" >
+<robot name="rover30" xmlns:xacro="http://ros.org/wiki/xacro" >
     <xacro:macro name="inertial_cylinder" params="mass length radius *origin">
         <inertial>

File: src2/rover30_description/urdf/lidar.xacro (robot description, xacro)
@@ -1,5 +1,5 @@
 <?xml version="1.0"?>
 <robot xmlns:xacro="http://ros.org/wiki/xacro" >
-    <xacro:include filename="interial_macros.xacro"/>
+    <xacro:include filename="$(find rover30_description)/urdf/interial_macros.xacro"/>
     <joint name="laser_joint" type="fixed">
         <parent link="base_link"/>
@@ -46,5 +46,5 @@
             <plugin name="laser_controller" filename="libgazebo_ros_ray_sensor.so">
                 <ros>
-                    <argument>~/out:=scan</argument>
+                    <argument>--ros-args --remap ~/out:=scan</argument>
                 </ros>
                 <output_type>sensor_msgs/LaserScan</output_type>

File: src2/rover30_description/urdf/rover30.urdf.xacro (robot description, xacro)
@@ -1,5 +1,6 @@
 <?xml version="1.0"?>
 <robot name="rover30" xmlns:xacro="http://ros.org/wiki/xacro">
-    <xacro:include filename="rover30_core.xacro"/>
-    <xacro:include filename="lidar.xacro"/>
+    <xacro:include filename="$(find rover30_description)/urdf/rover30_gz.xacro"/>
+    <xacro:include filename="$(find rover30_description)/urdf/rover30_core.xacro"/>
+    <xacro:include filename="$(find rover30_description)/urdf/lidar.xacro"/>
 </robot>

File: src2/rover30_description/urdf/rover30_core.xacro (robot description, xacro)
@@ -17,9 +17,9 @@
         <inertial>
             <origin xyz="0 0 0" rpy="0 0 0"/>
-            <mass value="20.0"/>
-            <inertia
-            ixx="1.0" ixy="1.0" ixz="1.0"
-            iyy="1.0" iyz="1.0"
-            izz="1.0" />
+            <mass value="100.0"/>
+            <inertia
+              ixx="10" ixy="10" ixz="10"
+              iyy="10" iyz="10"
+              izz="10"/>
         </inertial>
      </link>
@@ -44,7 +44,7 @@
             <mass value="2.0"/>
             <inertia
-              ixx="0.01" ixy="0.0" ixz="0.0"
-              iyy="0.01" iyz="0.0"
-              izz="0.01"/>
+              ixx="0.000002" ixy="-0.245562" ixz="0.969381"
+              iyy="0.001097" iyz="0.001097"
+              izz="-0.245562"/>
           </inertial>
     </link>
@@ -69,7 +69,7 @@
             <mass value="2.0"/>
             <inertia
-              ixx="0.01" ixy="0.0" ixz="0.0"
-              iyy="0.01" iyz="0.0"
-              izz="0.01"/>
+              ixx="0.000002" ixy="-0.245562" ixz="0.969381"
+              iyy="0.001097" iyz="0.001097"
+              izz="-0.245562"/>
           </inertial>
     </link>
@@ -94,7 +94,7 @@
             <mass value="2.0"/>
             <inertia
-              ixx="0.01" ixy="0.0" ixz="0.0"
-              iyy="0.01" iyz="0.0"
-              izz="0.01"/>
+              ixx="0.000002" ixy="-0.245562" ixz="0.969381"
+              iyy="0.001097" iyz="0.001097"
+              izz="-0.245562"/>
           </inertial>
     </link>
@@ -119,40 +119,108 @@
             <mass value="2.0"/>
             <inertia
-              ixx="0.01" ixy="0.0" ixz="0.0"
-              iyy="0.01" iyz="0.0"
-              izz="0.01"/>
+              ixx="0.000002" ixy="-0.245562" ixz="0.969381"
+              iyy="0.001097" iyz="0.001097"
+              izz="-0.245562"/>
           </inertial>
     </link>
     <link name="rfwOZ_link">
-        <visual>
-            <origin xyz="0 0 0" rpy="0 0 0"/>
-            <geometry>
-                <sphere radius="0.001"/>
-            </geometry>
-        </visual>
+            <visual>
+            <origin xyz="0 0 0" rpy="0 0 0"/>
+            <geometry>
+                  <cylinder radius="0.2" length="0.1"/>
+            </geometry>
+            <material name="green">
+                <color rgba="0.0 1.0 0.0 1.0"/>
+            </material>
+        </visual>
+        <collision>
+            <origin xyz="0 0 0" rpy="0 0 0"/>
+            <geometry>
+                 <cylinder radius="0.2" length="0.1"/>
+            </geometry>
+        </collision>
+        <inertial>
+            <origin xyz="0 0 0" rpy="0 0 0"/>
+            <mass value="2.0"/>
+            <inertia
+              ixx="0.01" ixy="0.0" ixz="0.0"
+              iyy="0.01" iyz="0.0"
+              izz="0.01"/>
+          </inertial>
     </link>
     <link name="lfwOZ_link">
-        <visual>
-            <origin xyz="0 0 0" rpy="0 0 0"/>
-            <geometry>
-                <sphere radius="0.001"/>
-            </geometry>
-        </visual>
+            <visual>
+            <origin xyz="0 0 0" rpy="0 0 0"/>
+            <geometry>
+                  <cylinder radius="0.2" length="0.1"/>
+            </geometry>
+            <material name="green">
+                <color rgba="0.0 1.0 0.0 1.0"/>
+            </material>
+        </visual>
+        <collision>
+            <origin xyz="0 0 0" rpy="0 0 0"/>
+            <geometry>
+                 <cylinder radius="0.2" length="0.1"/>
+            </geometry>
+        </collision>
+        <inertial>
+            <origin xyz="0 0 0" rpy="0 0 0"/>
+            <mass value="2.0"/>
+            <inertia
+              ixx="0.01" ixy="0.0" ixz="0.0"
+              iyy="0.01" iyz="0.0"
+              izz="0.01"/>
+          </inertial>
     </link>
     <link name="rrwOZ_link">
-        <visual>
-            <origin xyz="0 0 0" rpy="0 0 0"/>
-            <geometry>
-                <sphere radius="0.001"/>
-            </geometry>
-        </visual>
+            <visual>
+            <origin xyz="0 0 0" rpy="0 0 0"/>
+            <geometry>
+                  <cylinder radius="0.2" length="0.1"/>
+            </geometry>
+            <material name="green">
+                <color rgba="0.0 1.0 0.0 1.0"/>
+            </material>
+        </visual>
+        <collision>
+            <origin xyz="0 0 0" rpy="0 0 0"/>
+            <geometry>
+                 <cylinder radius="0.2" length="0.1"/>
+            </geometry>
+        </collision>
+        <inertial>
+            <origin xyz="0 0 0" rpy="0 0 0"/>
+            <mass value="2.0"/>
+            <inertia
+              ixx="0.01" ixy="0.0" ixz="0.0"
+              iyy="0.01" iyz="0.0"
+              izz="0.01"/>
+          </inertial>
     </link>
     <link name="lrwOZ_link">
-        <visual>
-            <origin xyz="0 0 0" rpy="0 0 0"/>
-            <geometry>
-                <sphere radius="0.001"/>
-            </geometry>
-        </visual>
+            <visual>
+            <origin xyz="0 0 0" rpy="0 0 0"/>
+            <geometry>
+                  <cylinder radius="0.2" length="0.1"/>
+            </geometry>
+            <material name="green">
+                <color rgba="0.0 1.0 0.0 1.0"/>
+            </material>
+        </visual>
+        <collision>
+            <origin xyz="0 0 0" rpy="0 0 0"/>
+            <geometry>
+                 <cylinder radius="0.2" length="0.1"/>
+            </geometry>
+        </collision>
+        <inertial>
+            <origin xyz="0 0 0" rpy="0 0 0"/>
+            <mass value="2.0"/>
+            <inertia
+              ixx="0.01" ixy="0.0" ixz="0.0"
+              iyy="0.01" iyz="0.0"
+              izz="0.01"/>
+          </inertial>
     </link>
      <joint name="base_joint" type="fixed">
